File: PCB/strawberryMacro.kicad_pcb (KiCad board)
At the start: 2 copper layers, 59.2 x 86 mm, 25 parts, among them SW1 SW_Push, SW10 RotaryEncoder, SW11 RotaryEncoder, SW2 SW_Push, SW3 SW_Push, SW4 SW_Push, SW5 SW_Push, SW6 SW_Push, SW7 SW_Push, SW8 SW_Push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

Commit message: Updated PCB
Parts:
- D1, D2, D3, D4, D5, D6, D7, D8, D9: footprint Diode_SMD:D_SOD-123 -> Diode_THT:D_DO-35_SOD27_P7.62mm_Horizontal
- moved D9 8.26 mm to (108.4, 93.4)
- moved D6 7.08 mm to (108.4, 72.7)
- moved D8 6.57 mm to (89.4, 93.4)
- moved D7 5.74 mm to (70.3, 93.2)
- moved D3 4.21 mm to (108.4, 53.9)
- moved D1 4.16 mm to (70.3, 55.2)
- moved D4 4.13 mm to (70.3, 72.6)
- moved D2 4.11 mm to (89.4, 54.9)
- moved D5 4.07 mm to (89.4, 72.8)
Routing:
- net Row 0: track 161.4 -> 96.5 mm, vias 2 -> 0
- net Column 2: track 147.0 -> 123.3 mm
- net Row 2: track 66.0 -> 55.0 mm, vias 5 -> 0
- net Row 1: track 80.6 -> 75.3 mm, vias 4 -> 0
- net Net-(D9-A): track 5.29 -> 4.46 mm
- net Net-(D1-A): track 5.23 -> 4.48 mm
- net Net-(D2-A): track 5.13 -> 4.52 mm
- net Net-(D4-A): track 4.55 -> 5.11 mm
- net Net-(D6-A): track 5.51 -> 4.97 mm
